File: Hardware/main_cj125.brd (EAGLE design)
At the start: 50 x 50 mm, 56 parts, among them IC1 CJ125_SOIC24, IC2 MEGA48/88/168-AU, IC3 REG1117_SOT-223, IC4 MCP6002SOIC, J1 AVR_SPI_PRG_6NS, T1 IRLR024NPBF

Commit message: Fixed names
Connections:
- new net NERNST: PAD6.P$1@1, PAD6.P$1@2
- net NERST: no longer PAD6.P$1@1, PAD6.P$1@2
Routing:
- net NERST: track 26.6 -> 21.0 mm
Changed lines of the file:
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@@
 </signal>
 <signal name="NERST">
-<contactref element="PAD6" pad="P$1@1"/>
 <contactref element="IC1" pad="2"/>
 <contactref element="R3" pad="2"/>
@@
 <wire x1="21.855" y1="11.06" x2="20.955" y2="10.16" width="0.3048" layer="1"/>
 <wire x1="20.955" y1="10.16" x2="20.955" y2="6.985" width="0.3048" layer="1"/>
-<contactref element="PAD6" pad="P$1@2"/>
-<wire x1="20.955" y1="6.985" x2="22.86" y2="5.08" width="0.3048" layer="1"/>
 <contactref element="R13" pad="1"/>
-<wire x1="22.86" y1="7.99" x2="22.86" y2="5.08" width="0.3048" layer="16"/>
+<wire x1="20.955" y1="6.985" x2="22.86" y2="7.99" width="0" layer="19" extent="1-16"/>
 </signal>
 <signal name="HEATER">
@@
 <wire x1="33.02" y1="41.275" x2="36.83" y2="45.085" width="0.3048" layer="16"/>
 </signal>
+<signal name="NERNST">
+<contactref element="PAD6" pad="P$1@1"/>
+<contactref element="PAD6" pad="P$1@2"/>
+</signal>
 </signals>
