File: Hardware/main_cj125.sch (EAGLE design)
At the start: 56 parts, among them IC1 CJ125_SOIC24, IC2 MEGA48/88/168-AU, IC3 REG1117_SOT-223, IC4 MCP6002SOIC, J1 AVR_SPI_PRG_6NS, T1 IRLR024NPBF

Commit message: Fixed names
Connections:
- new net NERNST: PAD6.P$1
- net NERST: no longer PAD6.P$1
Changed lines of the file:
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@@
 <net name="NERST" class="0">
-<segment>
-<wire x1="-48.26" y1="15.24" x2="-25.4" y2="15.24" width="0.1524" layer="91"/>
-<label x="-35.56" y="15.24" size="1.778" layer="95"/>
-<pinref part="PAD6" gate="A" pin="P$1"/>
-</segment>
 <segment>
 <pinref part="IC1" gate="G$1" pin="UN"/>
@@
 </segment>
 </net>
+<net name="NERNST" class="0">
+<segment>
+<wire x1="-48.26" y1="15.24" x2="-25.4" y2="15.24" width="0.1524" layer="91"/>
+<label x="-35.56" y="15.24" size="1.778" layer="95"/>
+<pinref part="PAD6" gate="A" pin="P$1"/>
+</segment>
+</net>
